File: docs/boarddesign/reveller-pi-B+HAT.sch (EAGLE design)
At the start: 23 parts, among them IC100 6581, Q100 IRF9Z24N, T100 BC547, X1 RASPI_BOARD_B+#_HDC, X101 PG203J, X102 CANTON-POWER

Commit message: Added box design and revised RevellerZero design
Raspberry Pi Rev B box design to allow for reveller HAT. Can be printed
with or without vented design. Designed in Solidworks 2016. RevellerZero
board design was revised due to CantonPower being placed slightly off
board.
Parts:
- added JUMPER: (no value), jumper:JP2W
Connections:
- net N$1 renamed 5VSTABIL
- new net CLKOC1: JUMPER.3, X1.GPIO13
- new net CLKRPI: JUMPER.1, X1.GPIO18
- new net PWCTLRPI: Q100.G, R105.1, X102-3.S
- net A0: now also X1.SPI_CE1
- net A1: now also X1.SPI_CE0
- net A2: now also X1.SPI_MISO
- net A3: now also X1.SPI_MOSI
- net A4: now also X1.SPI_SCLK
- net CLK: now also JUMPER.2; no longer X1.GPIO18
- net PWCTL: no longer Q100.G, R105.1, X102-3.S
